File: TopPCB/Top_rev1.sch (EAGLE design)
At the start: 0 parts

Commit message: added all components and connections for Top PCB.
Parts:
- added IC1: 74HC595D, 74xx-eu:74HC595D
- added JP1: (no value), SparkFun-Connectors:M06POGOPIN_HOLES_ONLY
- added R2, R3: (no value), SparkFun-Resistors:RESISTOR-ARRAY0603-ARV
- added U$1: 7-SEGMENT-DISPLAY-1"-RED, SparkFun-Displays:7-SEGMENT-DISPLAY-1"-RED
Connections:
- new net GND: IC1A.G, IC1A.QH*, JP1.1, U$1.G2
- new net INPUT+: JP1.3, U$1.G1
- new net N$1: R3D.2, U$1.DP
- new net N$10: IC1A.QE, R2D.1
- new net N$11: IC1A.QF, R2C.1
- new net N$12: IC1A.QG, R2B.1
- new net N$13: IC1A.QH, R2A.1
- new net N$14: R2C.2, U$1.A
- new net N$15: R2B.2, U$1.F
- new net N$16: R2A.2, U$1.G
- new net N$2: IC1A.QB, R3C.1
- new net N$3: R3C.2, U$1.E
- new net N$4: IC1A.QC, R3B.1
- new net N$5: IC1A.QD, R3A.1
- new net N$6: R3B.2, U$1.D
- new net N$7: R3A.2, U$1.C
- new net N$8: R2D.2, U$1.B
- new net N$9: IC1A.QA, R3D.1
- new net RCK: IC1A.RCK, JP1.5
- new net SCK: IC1A.SCK, JP1.4
- new net SERIAL: IC1A.SER, JP1.6
- new net VCC: IC1A.SCL, JP1.2
Other:
- note added: "1"
- note added: "Author: Zachary Nelson znelson1@ford.com"
